Commit message: ros_world

File: hubo_kart_display_v1/robots/drchubo_new_head.urdf (robot description, URDF)
Before this commit: robot hubo_kart_display_v1, 64 links, 63 joints
Links:
- removed link camera_c_link
- removed link camera_l_link
- removed link camera_r_link
- removed link head_base_link
- removed link lidar_optical_frame
- removed link lidar_tilt_link
- removed link ps_lower_base_link
- removed link ps_upper_base_link
- removed link turret_pan_link
- removed link turret_tilt_link
Joints:
- removed joint NKY
- removed joint camera_c
- removed joint camera_l
- removed joint camera_r
- removed joint lidar_optical_link
- removed joint lidar_tilt
- removed joint ps_lower_base
- removed joint ps_upper_base
- removed joint turret_pan
- removed joint turret_tilt
